File: TangNano20K-BaseBoard.kicad_pcb (KiCad board)
At the start: 2 copper layers, 0 parts

Commit message: Update schematic and start design pcb layout
Parts:
- added D1: LED, LED_SMD:LED_0805_2012Metric_Pad1.15x1.40mm_HandSolder, F.Cu at (161.6, 139.0)
- added D2: LED, LED_SMD:LED_0805_2012Metric_Pad1.15x1.40mm_HandSolder, F.Cu at (171.2, 139.0)
- added D3: LED, LED_SMD:LED_0805_2012Metric_Pad1.15x1.40mm_HandSolder, F.Cu at (181.0, 139.0)
- added D4: LED, LED_SMD:LED_0805_2012Metric_Pad1.15x1.40mm_HandSolder, F.Cu at (190.6, 139.0)
- added J1: Conn_01x20_Socket, Connector_PinSocket_2.54mm:PinSocket_1x20_P2.54mm_Vertical, F.Cu at (154.2, 95.8)
- added J2: Conn_01x20_Socket, Connector_PinSocket_2.54mm:PinSocket_1x20_P2.54mm_Vertical, F.Cu at (154.2, 78.0)
- added J3: Conn_01x06_Socket, Connector_PinSocket_2.54mm:PinSocket_1x06_P2.54mm_Vertical, F.Cu at (245.1, 99.3)
- added J4: Conn_01x06_Socket, Connector_PinSocket_2.54mm:PinSocket_1x06_P2.54mm_Vertical, F.Cu at (244.1, 135.3)
- added PB1: 1301.9315, MyFootPrints:13019319, F.Cu at (212.8, 124.4)
- added PB2: 1301.9315, MyFootPrints:13019319, F.Cu at (235.8, 124.4)
- added PB3: 1301.9315, MyFootPrints:13019319, F.Cu at (224.9, 112.2)
- added PB4: 1301.9315, MyFootPrints:13019319, F.Cu at (224.9, 136.6)
- added Q1: PN2222A, Package_TO_SOT_SMD:SOT-23, F.Cu at (168.5, 107.2)
- added Q2: PN2222A, Package_TO_SOT_SMD:SOT-23, F.Cu at (183.1, 107.0)
- added Q3: PN2222A, Package_TO_SOT_SMD:SOT-23, F.Cu at (188.5, 107.2)
- added Q4: PN2222A, Package_TO_SOT_SMD:SOT-23, F.Cu at (186.8, 132.1)
- added R1: 220R, Resistor_SMD:R_0805_2012Metric_Pad1.20x1.40mm_HandSolder, F.Cu at (173.1, 107.9)
- added R10: 330R, Resistor_SMD:R_0805_2012Metric_Pad1.20x1.40mm_HandSolder, F.Cu at (183.2, 103.5)
- added R11: 330R, Resistor_SMD:R_0805_2012Metric_Pad1.20x1.40mm_HandSolder, F.Cu at (188.7, 103.5)
- added R12: 330R, Resistor_SMD:R_0805_2012Metric_Pad1.20x1.40mm_HandSolder, F.Cu at (186.8, 136.9)
- added R13: 330R, Resistor_SMD:R_0805_2012Metric_Pad1.20x1.40mm_HandSolder, F.Cu at (163.9, 143.0)
- added R14: 330R, Resistor_SMD:R_0805_2012Metric_Pad1.20x1.40mm_HandSolder, F.Cu at (173.6, 143.0)
- added R15: 330R, Resistor_SMD:R_0805_2012Metric_Pad1.20x1.40mm_HandSolder, F.Cu at (183.3, 143.0)
- added R16: 330R, Resistor_SMD:R_0805_2012Metric_Pad1.20x1.40mm_HandSolder, F.Cu at (193.1, 143.0)
- added R19: 10k, Resistor_SMD:R_0805_2012Metric_Pad1.20x1.40mm_HandSolder, F.Cu at (159.0, 143.0)
- added R2: 220R, Resistor_SMD:R_0805_2012Metric_Pad1.20x1.40mm_HandSolder, F.Cu at (193.4, 107.5)
- added R20: 10k, Resistor_SMD:R_0805_2012Metric_Pad1.20x1.40mm_HandSolder, F.Cu at (168.8, 143.0)
- added R21: 10k, Resistor_SMD:R_0805_2012Metric_Pad1.20x1.40mm_HandSolder, F.Cu at (178.5, 143.0)
- added R22: 10k, Resistor_SMD:R_0805_2012Metric_Pad1.20x1.40mm_HandSolder, F.Cu at (188.2, 143.0)
- added R23: 10k, Resistor_SMD:R_0805_2012Metric_Pad1.20x1.40mm_HandSolder, F.Cu at (214.9, 131.2)
- added R24: 10k, Resistor_SMD:R_0805_2012Metric_Pad1.20x1.40mm_HandSolder, F.Cu at (235.7, 131.0)
- added R25: 10k, Resistor_SMD:R_0805_2012Metric_Pad1.20x1.40mm_HandSolder, F.Cu at (214.5, 118.6)
- added R26: 10k, Resistor_SMD:R_0805_2012Metric_Pad1.20x1.40mm_HandSolder, F.Cu at (235.7, 119.0)
- added R27: 10k, Resistor_SMD:R_0805_2012Metric_Pad1.20x1.40mm_HandSolder, F.Cu at (239.8, 77.9)
- added R28: 10k, Resistor_SMD:R_0805_2012Metric_Pad1.20x1.40mm_HandSolder, F.Cu at (244.9, 77.9)
- added R3: 220R, Resistor_SMD:R_0805_2012Metric_Pad1.20x1.40mm_HandSolder, F.Cu at (176.9, 132.2)
- added R4: 220R, Resistor_SMD:R_0805_2012Metric_Pad1.20x1.40mm_HandSolder, F.Cu at (168.2, 132.2)
- added R5: 220R, Resistor_SMD:R_0805_2012Metric_Pad1.20x1.40mm_HandSolder, F.Cu at (163.9, 132.2)
- added R6: 220R, Resistor_SMD:R_0805_2012Metric_Pad1.20x1.40mm_HandSolder, F.Cu at (177.5, 107.9)
- added R7: 220R, Resistor_SMD:R_0805_2012Metric_Pad1.20x1.40mm_HandSolder, F.Cu at (181.2, 132.2)
- added R8: 220R, Resistor_SMD:R_0805_2012Metric_Pad1.20x1.40mm_HandSolder, F.Cu at (172.5, 132.2)
- added R9: 330R, Resistor_SMD:R_0805_2012Metric_Pad1.20x1.40mm_HandSolder, F.Cu at (168.4, 103.5)
- added SW1: SW_SPDT_321, MyFootPrints:SL19121, F.Cu at (161.5, 156.4)
- added SW2: SW_SPDT_321, MyFootPrints:SL19121, F.Cu at (171.2, 156.4)
- added SW3: SW_SPDT_321, MyFootPrints:SL19121, F.Cu at (180.9, 156.4)
- added SW4: SW_SPDT_321, MyFootPrints:SL19121, F.Cu at (190.6, 156.4)
- added SW5: SW_SPDT_321, MyFootPrints:SL19121, F.Cu at (242.4, 92.2)
- added U1: CC56-12EWA, Display_7Segment:CA56-12EWA, F.Cu at (172.0, 127.2)
- added U2: SSD1306, MyFootPrints:128x64OLED, F.Cu at (222.0, 88.1)
Other:
- board outline added: 100 x 85 mm
