File: TangNano20K-BaseBoard.kicad_pcb (KiCad board)
At the start: 2 copper layers, 100 x 100 mm, 48 parts, among them J1 Conn_01x20_Socket, J2 Conn_01x20_Socket, J3 Conn_02x06_Odd_Even, Q1 PN2222A, Q2 PN2222A, Q3 PN2222A, Q4 PN2222A, SW1 SW_SPDT_321, SW2 SW_SPDT_321, SW3 SW_SPDT_321, SW4 SW_SPDT_321, SW5 SW_SPDT_321, U1 CC56-12EWA, U2 SSD1306

Commit message: Update PCB
Parts:
- moved J2 3.03 mm to (175.9, 112.8)
- moved J1 3.03 mm to (175.9, 130.5)
- moved PB1 1.16 mm to (208.0, 147.8)
- moved PB2 1.16 mm to (224.9, 147.8)
- moved PB3 1.16 mm to (208.0, 161.0)
- moved PB4 1.16 mm to (224.9, 161.0)
- moved R23 1.16 mm to (201.9, 141.9)
- moved R24 1.16 mm to (218.8, 141.9)
- moved R25 1.16 mm to (201.8, 155.0)
- moved R26 1.16 mm to (218.8, 154.9)
- moved R2 0.78 mm to (192.7, 77.2)
- moved J3 0.32 mm to (236.9, 160.9)
- moved R10 0.23 mm to (181.0, 73.1)
Connections:
- J3 pad 10: /53 -> /30
- J3 pad 11: /49 -> /72
- J3 pad 12: /52 -> /31
- J3 pad 5: /80 -> /15
- J3 pad 6: /86 -> /26
- J3 pad 7: /41 -> /16
- J3 pad 8: /79 -> /29
- J3 pad 9: /55 -> /71
- PB1 pad 4: /75 -> /77
- PB2 pad 4: /76 -> /27
- PB3 pad 4: /77 -> /28
- PB4 pad 4: /85 -> /25
- R1 pad 1: /27 -> /48
- R10 pad 2: /54 -> /49
- R11 pad 2: /51 -> /86
- R12 pad 2: /48 -> /54
- R13 pad 1: /15 -> /17
- R14 pad 1: /16 -> /20
- R15 pad 1: /17 -> /19
- R19 pad 2: /71 -> /73
- R2 pad 1: /28 -> /79
- R20 pad 2: /72 -> /74
- R21 pad 2: /73 -> /75
- R22 pad 2: /74 -> /85
- R23 pad 2: /75 -> /77
- R24 pad 2: /76 -> /27
- R25 pad 2: /77 -> /28
- R26 pad 2: /85 -> /25
- R27 pad 2: /19 -> /53
- R28 pad 1: /20 -> /52
- R3 pad 1: /25 -> /41
- R4 pad 1: /26 -> /80
- R5 pad 1: /29 -> /76
- R6 pad 1: /30 -> /55
- R7 pad 1: /31 -> /56
- R9 pad 2: /56 -> /51
- SW1 pad 1: /71 -> /73
- SW2 pad 1: /72 -> /74
- SW3 pad 1: /73 -> /75
- SW4 pad 1: /74 -> /85
- U2 pad 3: /19 -> /53
- U2 pad 4: /20 -> /52
Other:
- board text added: "3V3"
- board text added: "GND"

Commit message: Update PCB
Parts:
- moved R2 3.95 mm to (188.7, 77.1), turned to 180 degrees
- moved Q3 2.62 mm to (184.4, 76.7)
- moved R11 2.62 mm to (184.4, 73.1)
- moved R1 0.83 mm to (171.5, 77.1)
- moved Q2 0.83 mm to (180.2, 76.7)
- moved R10 0.83 mm to (180.2, 73.1)
- moved R6 0.83 mm to (176.0, 77.1)
- moved Q1 0.43 mm to (167.4, 76.7)
- moved R9 0.43 mm to (167.4, 73.1)
Other:
- board text added: "OLED on/off"
Changed lines of the file:
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@@
 	(footprint "Package_TO_SOT_SMD:SOT-23"
 		(layer "F.Cu")
-		(at 187 76.7275 -90)
+		(at 184.378908 76.651746 -90)
 		(descr "SOT, 3 Pin (JEDEC TO-236 Var AB https://www.jedec.org/document_search?search_api_views_fulltext=TO-236)")
 		(tags "SOT TO_SOT_SMD")
 		(property "Reference" "Q3"
-			(at 0 -2.4 90)
+			(at -0.001723 -2.454556 90)
 			(layer "F.SilkS")
+			(hide yes)
 			(effects
 				(font
@@
 	(footprint "Resistor_SMD:R_0805_2012Metric_Pad1.20x1.40mm_HandSolder"
 		(layer "F.Cu")
-		(at 167.02 73.14)
+		(at 167.446794 73.0666)
 		(descr "Resistor SMD 0805 (2012 Metric), square (rectangular) end terminal, IPC-7351 nominal with elongated pad for handsoldering. (Body size source: IPC-SM-782 page 72, https://www.pcb-3d.com/wordpress/wp-content/uploads/ipc-sm-782a_amendment_1_and_2.pdf)")
 		(tags "resistor handsolder")
@@
 	(footprint "Resistor_SMD:R_0805_2012Metric_Pad1.20x1.40mm_HandSolder"
 		(layer "F.Cu")
-		(at 176.78 77.2)
+		(at 175.956794 77.1266)
 		(descr "Resistor SMD 0805 (2012 Metric), square (rectangular) end terminal, IPC-7351 nominal with elongated pad for handsoldering. (Body size source: IPC-SM-782 page 72, https://www.pcb-3d.com/wordpress/wp-content/uploads/ipc-sm-782a_amendment_1_and_2.pdf)")
 		(tags "resistor handsolder")
 		(property "Reference" "R6"
-			(at -0.016 -1.778 0)
+			(at -0.016 -1.65 0)
 			(layer "F.SilkS")
 			(effects
@@
 	(footprint "Package_TO_SOT_SMD:SOT-23"
 		(layer "F.Cu")
-		(at 166.96 76.7275 -90)
+		(at 167.386794 76.6541 -90)
 		(descr "SOT, 3 Pin (JEDEC TO-236 Var AB https://www.jedec.org/document_search?search_api_views_fulltext=TO-236)")
 		(tags "SOT TO_SOT_SMD")
 		(property "Reference" "Q1"
-			(at 0 -2.4 90)
+			(at 0 -2.47 90)
 			(layer "F.SilkS")
+			(hide yes)
 			(effects
 				(font
@@
 	(footprint "Package_TO_SOT_SMD:SOT-23"
 		(layer "F.Cu")
-		(at 180.99 76.7275 -90)
+		(at 180.166794 76.6541 -90)
 		(descr "SOT, 3 Pin (JEDEC TO-236 Var AB https://www.jedec.org/document_search?search_api_views_fulltext=TO-236)")
 		(tags "SOT TO_SOT_SMD")
 		(property "Reference" "Q2"
-			(at 0 -2.4 90)
+			(at 0 -2.45 90)
 			(layer "F.SilkS")
+			(hide yes)
 			(effects
 				(font
@@
 	(footprint "Resistor_SMD:R_0805_2012Metric_Pad1.20x1.40mm_HandSolder"
 		(layer "F.Cu")
-		(at 180.99 73.14)
+		(at 180.166794 73.0666)
 		(descr "Resistor SMD 0805 (2012 Metric), square (rectangular) end terminal, IPC-7351 nominal with elongated pad for handsoldering. (Body size source: IPC-SM-782 page 72, https://www.pcb-3d.com/wordpress/wp-content/uploads/ipc-sm-782a_amendment_1_and_2.pdf)")
 		(tags "resistor handsolder")
 		(property "Reference" "R10"
-			(at 0 -2.032 0)
+			(at 0 -1.65 0)
 			(layer "F.SilkS")
 			(effects
@@
 	(footprint "Resistor_SMD:R_0805_2012Metric_Pad1.20x1.40mm_HandSolder"
 		(layer "F.Cu")
-		(at 192.65 77.2)
+		(at 188.698908 77.124246 180)
 		(descr "Resistor SMD 0805 (2012 Metric), square (rectangular) end terminal, IPC-7351 nominal with elongated pad for handsoldering. (Body size source: IPC-SM-782 page 72, https://www.pcb-3d.com/wordpress/wp-content/uploads/ipc-sm-782a_amendment_1_and_2.pdf)")
 		(tags "resistor handsolder")
 		(property "Reference" "R2"
-			(at 0 -1.65 0)
+			(at 0 1.65 0)
 			(layer "F.SilkS")
 			(effects
@@
 		(duplicate_pad_numbers_are_jumpers no)
 		(fp_line
-			(start -0.227064 -0.735)
-			(end 0.227064 -0.735)
+			(start -0.227064 0.735)
+			(end 0.227064 0.735)
 			(stroke
 				(width 0.12)
@@
 		)
 		(fp_line
-			(start -0.227064 0.735)
-			(end 0.227064 0.735)
+			(start -0.227064 -0.735)
+			(end 0.227064 -0.735)
 			(stroke
 				(width 0.12)
@@
 		)
 		(pad "1" smd roundrect
-			(at -1 0)
+			(at -1 0 180)
 			(size 1.2 1.4)
 			(layers "F.Cu" "F.Mask" "F.Paste")
@@
 		)
 		(pad "2" smd roundrect
-			(at 1 0)
+			(at 1 0 180)
 			(size 1.2 1.4)
 			(layers "F.Cu" "F.Mask" "F.Paste")
@@
 	(footprint "Resistor_SMD:R_0805_2012Metric_Pad1.20x1.40mm_HandSolder"
 		(layer "F.Cu")
-		(at 187 73.14)
+		(at 184.378908 73.064246)
 		(descr "Resistor SMD 0805 (2012 Metric), square (rectangular) end terminal, IPC-7351 nominal with elongated pad for handsoldering. (Body size source: IPC-SM-782 page 72, https://www.pcb-3d.com/wordpress/wp-content/uploads/ipc-sm-782a_amendment_1_and_2.pdf)")
 		(tags "resistor handsolder")
@@
 	(footprint "Resistor_SMD:R_0805_2012Metric_Pad1.20x1.40mm_HandSolder"
 		(layer "F.Cu")
-		(at 172.36 77.2)
+		(at 171.536794 77.1266)
 		(descr "Resistor SMD 0805 (2012 Metric), square (rectangular) end terminal, IPC-7351 nominal with elongated pad for handsoldering. (Body size source: IPC-SM-782 page 72, https://www.pcb-3d.com/wordpress/wp-content/uploads/ipc-sm-782a_amendment_1_and_2.pdf)")
 		(tags "resistor handsolder")
@@
 		(layer "F.SilkS")
 		(effects
+			(font
+				(size 1 1)
+				(thickness 0.15)
+			)
+		)
+	)
+	(gr_text "OLED on/off"
+		(at 242.5 94.89 0)
+		(layer "F.SilkS")
+		(effects

Commit message: Update pcb
Parts:
- added J4: Conn_02x03_Odd, Connector_PinSocket_2.54mm:PinSocket_2x03_P2.54mm_Horizontal, F.Cu at (213.1, 87.1)
- moved D1 101.6 mm to (259.2, 120.3)
- moved R13 100.0 mm to (259.2, 122.4)
- moved D2 97.1 mm to (264.2, 120.3)
- moved R14 95.5 mm to (264.1, 122.4)
- moved D3 92.5 mm to (269.2, 120.3)
- moved R15 91.0 mm to (269.2, 122.4)
- moved D4 88.0 mm to (274.2, 120.3)
- moved R16 86.5 mm to (274.1, 122.4)
- moved R9 70.9 mm to (236.3, 89.9), turned to 180 degrees
- moved Q1 69.7 mm to (236.3, 86.5), turned to 90 degrees
- moved R21 69.0 mm to (221.6, 122.5), turned to 90 degrees
- moved R1 68.8 mm to (239.7, 86.6), turned to 90 degrees
- moved R10 67.3 mm to (245.3, 89.9), turned to 180 degrees
- moved R11 67.1 mm to (249.3, 89.9), turned to 180 degrees
- moved R6 66.7 mm to (242.0, 86.6), turned to 90 degrees
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- renumbered R23 to R17, R24 to R18, R25 to R19, R26 to R20, R19 to R21, R20 to R22, R21 to R23, R22 to R24, R27 to R25, R28 to R26
Connections:
- J3 pad 10: /30 -> /29
- J3 pad 11: /72 -> /25
- J3 pad 12: /31 -> /26
- J3 pad 5: /15 -> /16
- J3 pad 6: /26 -> /31
- J3 pad 7: /16 -> /27
- J3 pad 8: /29 -> /30
- J3 pad 9: /71 -> /28
- PB1 pad 4: /77 -> /85
- PB2 pad 4: /27 -> /15
- PB3 pad 4: /28 -> /75
- PB4 pad 4: /25 -> /77
- R17 pad 2: /77 -> /85
- R18 pad 2: /27 -> /15
- R19 pad 2: /28 -> /75
- R20 pad 2: /25 -> /77
- R21 pad 2: /73 -> /72
- R22 pad 2: /74 -> /71
- R23 pad 2: /75 -> /73
- R24 pad 2: /85 -> /74
- SW1 pad 1: /73 -> /72
- SW2 pad 1: /74 -> /71
- SW3 pad 1: /75 -> /73
- SW4 pad 1: /85 -> /74
Routing:
- net +3V3: track 0.00 -> 268.9 mm, vias 0 -> 1
- net Net-(SW5-C): track 0.00 -> 87.7 mm
- net /72: track 0.00 -> 84.6 mm
- net /71: track 0.00 -> 75.9 mm
- net /16: track 0.00 -> 63.7 mm
- net /27: track 0.00 -> 59.1 mm
- net /31: track 0.00 -> 57.4 mm
- net /28: track 0.00 -> 54.5 mm
- net /30: track 0.00 -> 53.8 mm
- net /77: track 0.00 -> 52.9 mm
- net /29: track 0.00 -> 51.9 mm
- net /26: track 0.00 -> 50.5 mm
- net /25: track 0.00 -> 49.8 mm
- net /15: track 0.00 -> 42.3 mm
- net /75: track 0.00 -> 40.8 mm
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- added copper zone on B.Cu, net GND
- added copper zone on F.Cu, net GND
Other:
- board size 100 x 100 mm -> 100 x 90 mm
- board text added: "16|31"
- board text added: "25|26"
- board text added: "27|30"
- board text added: "28|29"
- board text added: "5V"
- board text added: "HDMI"
- board text added: "Michał Głuszak"
- board text added: "Tang Nano 20K"
- board text added: "TangNano20K-BaseBoard"
- board text added: "USB-C"
- board text removed: "Q4"
